Commit message: env: Modify humble to iron.

File: src/robot_dsc/urdf/diff_drive.urdf.xacro (robot description, xacro)
@@ -1,4 +1,5 @@
 <?xml version="1.0"?>
-<robot xmlns:xacro="http://www.ros.org/wiki/xacro" name="simple_dd_bot">
+<robot xmlns:xacro="http://www.ros.org/wiki/xacro" name="simple_dd_bot_v2">
+    <!-- Properties (保持不变) -->
     <xacro:property name="base_width" value="0.2"/>
     <xacro:property name="base_length" value="0.3"/>
@@ -8,130 +9,105 @@
     <xacro:property name="wheel_offset_y" value="${base_width/2 + wheel_thickness/2}"/>
     <xacro:property name="wheel_offset_z" value="${-base_height/2 + wheel_radius}"/>
+    <xacro:property name="camera_link_size" value="0.02"/>
+    <!-- Inertia Macros (保持不变) -->
+    <xacro:macro name="box_inertia" params="m x y z">
+        <inertia ixx="${m*(y*y+z*z)/12}" ixy="0" ixz="0" iyy="${m*(x*x+z*z)/12}" iyz="0" izz="${m*(x*x+y*y)/12}"/>
+    </xacro:macro>
+    <xacro:macro name="cylinder_inertia" params="m r h">
+        <inertia ixx="${m*(3*r*r+h*h)/12}" ixy="0" ixz="0" iyy="${m*(3*r*r+h*h)/12}" iyz="0" izz="${m*r*r/2}"/>
+    </xacro:macro>
+    <xacro:macro name="sphere_inertia" params="m r">
+        <inertia ixx="${2*m*r*r/5}" ixy="0" ixz="0" iyy="${2*m*r*r/5}" iyz="0" izz="${2*m*r*r/5}"/>
+    </xacro:macro>
+    <!-- Base Link -->
     <link name="base_link">
-        <visual>
-            <geometry>
-                <box size="${base_length} ${base_width} ${base_height}"/>
-            </geometry>
-            <material name="grey">
-                <color rgba="0.5 0.5 0.5 1"/>
-            </material>
-        </visual>
-        <collision>
-            <geometry>
-                <box size="${base_length} ${base_width} ${base_height}"/>
-            </geometry>
-        </collision>
-        <inertial> <!-- 简化惯性 -->
-            <mass value="1.0"/>
-            <inertia ixx="0.01" ixy="0" ixz="0" iyy="0.01" iyz="0" izz="0.01"/>
-        </inertial>
+        <visual><geometry><box size="${base_length} ${base_width} ${base_height}"/></geometry><material name="grey"><color rgba="0.5 0.5 0.5 1"/></material></visual>
+        <collision><geometry><box size="${base_length} ${base_width} ${base_height}"/></geometry></collision>
+        <inertial><mass value="1.0"/><xacro:box_inertia m="1.0" x="${base_length}" y="${base_width}" z="${base_height}"/></inertial>
     </link>
+    <!-- Wheels Macro -->
     <xacro:macro name="wheel_link" params="prefix reflect_y">
         <link name="${prefix}_wheel_link">
-            <visual>
-                <origin xyz="0 0 0" rpy="${pi/2} 0 0"/>
-                <geometry>
-                    <cylinder radius="${wheel_radius}" length="${wheel_thickness}"/>
-                </geometry>
-                <material name="black">
-                    <color rgba="0.1 0.1 0.1 1"/>
-                </material>
-            </visual>
+            <visual><origin xyz="0 0 0" rpy="${pi/2} 0 0"/><geometry><cylinder radius="${wheel_radius}" length="${wheel_thickness}"/></geometry><material name="black"><color rgba="0.1 0.1 0.1 1"/></material></visual>
             <collision>
                 <origin xyz="0 0 0" rpy="${pi/2} 0 0"/>
-                <geometry>
-                    <cylinder radius="${wheel_radius}" length="${wheel_thickness}"/>
-                </geometry>
+                <geometry><cylinder radius="${wheel_radius}" length="${wheel_thickness}"/></geometry>
+                <!-- FIX 1: 为驱动轮添加摩擦力 -->
+                <surface>
+                    <friction>
+                        <ode>
+                            <mu>1.0</mu>
+                            <mu2>1.0</mu2>
+                        </ode>
+                    </friction>
+                </surface>
             </collision>
-            <inertial> <!-- 简化惯性 -->
-                <mass value="0.1"/>
-                <inertia ixx="0.001" ixy="0" ixz="0" iyy="0.001" iyz="0" izz="0.001"/>
-            </inertial>
+            <inertial><mass value="0.1"/><origin xyz="0 0 0" rpy="${pi/2} 0 0"/><xacro:cylinder_inertia m="0.1" r="${wheel_radius}" h="${wheel_thickness}"/></inertial>
         </link>
         <joint name="${prefix}_wheel_joint" type="continuous">
-            <parent link="base_link"/>
-            <child link="${prefix}_wheel_link"/>
-            <origin xyz="0 ${reflect_y * wheel_offset_y} ${wheel_offset_z}" rpy="0 0 0"/>
-            <axis xyz="0 1 0"/>
+            <parent link="base_link"/><child link="${prefix}_wheel_link"/><origin xyz="0 ${reflect_y * wheel_offset_y} ${wheel_offset_z}" rpy="0 0 0"/><axis xyz="0 1 0"/>
         </joint>
     </xacro:macro>
     <xacro:wheel_link prefix="left" reflect_y="1"/>
     <xacro:wheel_link prefix="right" reflect_y="-1"/>
-    <!-- 简单的摄像头 -->
-    <xacro:property name="camera_link_size" value="0.02"/>
+    <!-- FIX 2: 移除独立的caster link和joint，直接在Gazebo中定义 -->
+    <!-- 原来的caster link和joint已被删除 -->
+    <!-- Camera Link & Joint -->
     <link name="camera_link">
-        <visual>
-            <geometry>
-                <box size="${camera_link_size} ${camera_link_size} ${camera_link_size}"/>
-            </geometry>
-            <material name="blue">
-                <color rgba="0 0 1 1"/>
-            </material>
-        </visual>
-        <collision>
-            <geometry>
-                <box size="${camera_link_size} ${camera_link_size} ${camera_link_size}"/>
-            </geometry>
-        </collision>
-        <inertial>
-            <mass value="0.01"/>
-            <inertia ixx="1e-6" ixy="0" ixz="0" iyy="1e-6" iyz="0" izz="1e-6"/>
-        </inertial>
+        <inertial><mass value="0.01"/><xacro:box_inertia m="0.01" x="0.01" y="0.01" z="0.01"/></inertial>
     </link>
     <joint name="camera_joint" type="fixed">
         <parent link="base_link"/>
         <child link="camera_link"/>
-        <origin xyz="${base_length/2 - camera_link_size/2} 0 ${base_height/2}" rpy="0 0 0"/>
+        <origin xyz="${base_length/2 - 0.01} 0 ${base_height/2}" rpy="0 0.52 0"/>
     </joint>
-    <!-- Gazebo Plugins -->
+    <!-- =================================================================== -->
+    <!-- ================ Gazebo Sim (New Gazebo) Integration ================ -->
+    <!-- =================================================================== -->
+    <!-- Gazebo插件和物理属性定义 -->
     <gazebo>
-        <plugin name="gazebo_ros_diff_drive" filename="libgazebo_ros_diff_drive.so">
-            <ros>
-                <namespace>/robot</namespace>
-            </ros>
-            <update_rate>30</update_rate>
-            <!-- Wheels -->
+        <!-- 差分驱动插件 (保持不变) -->
+        <plugin filename="gz-sim-diff-drive-system" name="gz::sim::systems::DiffDrive">
             <left_joint>left_wheel_joint</left_joint>
             <right_joint>right_wheel_joint</right_joint>
-            <!-- Kinematics -->
-            <wheel_separation>${base_width + wheel_thickness}</wheel_separation> <!-- 估算轮距 -->
-            <wheel_diameter>${2*wheel_radius}</wheel_diameter>
-            <!-- Odometry -->
-            <odometry_frame>odom</odometry_frame>
-            <robot_base_frame>base_link</robot_base_frame>
-            <publish_odom>true</publish_odom>
-            <publish_odom_tf>true</publish_odom_tf>
-            <publish_wheel_tf>false</publish_wheel_tf>
-            <!-- Topic names -->
-            <command_topic>cmd_vel</command_topic>
-            <odometry_topic>odom</odometry_topic>
+            <wheel_separation>${base_width + wheel_thickness}</wheel_separation>
+            <wheel_radius>${wheel_radius}</wheel_radius>
+            <topic>/cmd_vel</topic>
+            <odom_topic>/odom</odom_topic>
+            <tf_topic>/tf</tf_topic>
         </plugin>
     </gazebo>
+    <!-- FIX 2: 在base_link上直接定义一个无摩擦的球形碰撞体作为caster -->
+    <gazebo reference="base_link">
+        <collision name="caster_collision">
+            <pose>${base_length/2 * 0.8} 0 ${-base_height/2 + 0.025} 0 0 0</pose>
+            <geometry><sphere><radius>0.025</radius></sphere></geometry>
+            <surface>
+                <friction><ode><mu>0.0</mu><mu2>0.0</mu2></ode></friction>
+            </surface>
+        </collision>
+        <material>Gazebo/Grey</material>
+    </gazebo>
     <gazebo reference="camera_link">
-        <sensor name="camera_sensor" type="camera">
-            <update_rate>10.0</update_rate>
-            <camera name="head_camera">
-                <horizontal_fov>1.047</horizontal_fov> <!-- 约60度 -->
-                <image>
-                    <width>320</width>
-                    <height>240</height>
-                    <format>R8G8B8</format>
-                </image>
-                <clip>
-                    <near>0.05</near>
-                    <far>8.0</far>
-                </clip>
+        <!-- a) RGB摄像头 -->
+        <sensor name="rgb_camera_sensor" type="camera">
+            <update_rate>20.0</update_rate>
+            <camera>
+                <horizontal_fov>1.047</horizontal_fov>
+                <image><width>640</width><height>480</height><format>R8G8B8</format></image>
+                <clip><near>0.05</near><far>8.0</far></clip>
             </camera>
-            <plugin name="camera_controller" filename="libgazebo_ros_camera.so">
-                <ros>
-                    <namespace>/my_robot</namespace>
-                    <argument>--ros-args --remap __node:=camera_driver_node</argument>
-                    <argument>--ros-args --remap /my_robot/camera_sensor/image_raw:=/my_robot/camera/image_raw</argument>
-                    <argument>--ros-args --remap /my_robot/camera_sensor/camera_info:=/my_robot/camera/camera_info</argument>
-                </ros>
-                <camera_name>camera_sensor</camera_name>
-                <frame_name>camera_link</frame_name>
-                <hack_baseline>0.0</hack_baseline> <!-- 对于单目相机 -->
-            </plugin>
+            <topic>rgb_camera</topic>
+            <visualize>true</visualize>
+        </sensor>
+        <sensor name="semantic_camera_sensor" type="semantic_segmentation_camera">
+            <update_rate>20.0</update_rate>
+            <camera>
+                <horizontal_fov>1.047</horizontal_fov>
+                <image><width>640</width><height>480</height></image>
+                <clip><near>0.05</near><far>8.0</far></clip>
+            </camera>
+            <topic>semantic_camera</topic>
+            <visualize>true</visualize>
         </sensor>
     </gazebo>

Commit message: fix: Fix base_link.

File: src/robot_dsc/urdf/diff_drive.urdf.xacro (robot description, xacro)
@@ -20,4 +20,10 @@
         <inertia ixx="${2*m*r*r/5}" ixy="0" ixz="0" iyy="${2*m*r*r/5}" iyz="0" izz="${2*m*r*r/5}"/>
     </xacro:macro>
+    <link name="base_footprint"/>
+    <joint name="base_footprint_to_base_link_joint" type="fixed">
+        <parent link="base_footprint"/>
+        <child link="base_link"/>
+        <origin xyz="0 0 0" rpy="0 0 0"/>
+    </joint>
     <!-- Base Link -->
     <link name="base_link">
@@ -99,7 +105,12 @@
             </camera>
             <topic>rgb_camera</topic>
+            <always_on>1</always_on>
             <visualize>true</visualize>
+            <!-- 添加这个插件 -->
+            <!-- plugin name="gz::sim::systems::Camera" filename="gz-sim-camera-system">
+                <topic>rgb_camera</topic>
+            </plugin -->
         </sensor>
-        <sensor name="semantic_camera_sensor" type="semantic_segmentation_camera">
+        <sensor name="semantic_camera_sensor" type="segmentation">
             <update_rate>20.0</update_rate>
             <camera>
@@ -108,6 +119,10 @@
                 <clip><near>0.05</near><far>8.0</far></clip>
             </camera>
-            <topic>semantic_camera</topic>
+            <topic>/semantic_camera</topic>
+            <always_on>1</always_on>
             <visualize>true</visualize>
+            <!-- plugin name="gz::sim::systems::SegmentationCamera" filename="gz-sim-segmentation-camera-system">
+                <topic>/semantic_camera</topic>
+            </plugin -->
         </sensor>
     </gazebo>

Commit message: feat: Add the avoidance policy.

File: src/robot_dsc/urdf/diff_drive.urdf.xacro (robot description, xacro)
@@ -68,4 +68,25 @@
         <origin xyz="${base_length/2 - 0.01} 0 ${base_height/2}" rpy="0 0.52 0"/>
     </joint>
+    <!-- 创建一个用于放置LIDAR的link -->
+    <link name="lidar_link">
+        <inertial>
+            <mass value="0.1"/>
+            <xacro:box_inertia m="0.1" x="0.05" y="0.05" z="0.05"/>
+        </inertial>
+        <visual>
+            <geometry><box size="0.05 0.05 0.05"/></geometry>
+            <material name="blue"><color rgba="0 0 1 1"/></material>
+        </visual>
+        <collision>
+            <geometry><box size="0.05 0.05 0.05"/></geometry>
+        </collision>
+    </link>
+    <!-- 将LIDAR link固定在base_link的前方 -->
+    <joint name="lidar_joint" type="fixed">
+        <parent link="base_link"/>
+        <child link="lidar_link"/>
+        <!-- 放置在车体最前端、略高于车体的位置 -->
+        <origin xyz="${base_length/2} 0 ${base_height/2 + 0.025}" rpy="0 0 0"/>
+    </joint>
     <!-- =================================================================== -->
     <!-- ================ Gazebo Sim (New Gazebo) Integration ================ -->
@@ -129,3 +150,34 @@
         </sensor>
     </gazebo>
+    <!-- Gazebo传感器定义 -->
+    <gazebo reference="lidar_link">
+        <!-- 添加LIDAR传感器插件 -->
+        <sensor name="gpu_lidar" type="gpu_ray">
+            <pose>0 0 0 0 0 0</pose>
+            <visualize>true</visualize> <!-- 在Gazebo中显示激光线 -->
+            <update_rate>10</update_rate>
+            <ray>
+                <scan>
+                    <horizontal>
+                        <samples>360</samples> <!-- 360条激光线 -->
+                        <resolution>1</resolution>
+                        <min_angle>-2.35619</min_angle> <!-- -135度 -->
+                        <max_angle>2.35619</max_angle>  <!-- +135度 -->
+                    </horizontal>
+                </scan>
+                <range>
+                    <min>0.1</min> <!-- 最小探测距离 -->
+                    <max>10.0</max> <!-- 最大探测距离 -->
+                    <resolution>0.01</resolution>
+                </range>
+                <noise>
+                    <type>gaussian</type>
+                    <mean>0.0</mean>
+                    <stddev>0.01</stddev>
+                </noise>
+            </ray>
+            <topic>/scan</topic> <!-- ROS话题名 -->
+            <frame>lidar_link</frame>
+        </sensor>
+    </gazebo>
 </robot>
